Commit message: update

File: urdf/simple_box.urdf (robot description, URDF)
Before this commit: robot simple_box, 1 links, 0 joints
Links:
- link box_link: mass 0.6 -> 0.3; geometry collision box size=0.3 0.3 0.3; visual box size=0.3 0.3 0.3

Commit message: update

File: urdf/simple_box.urdf (robot description, URDF)
Before this commit: robot simple_box, 1 links, 0 joints
Links:
- link box_link: geometry collision box size=0.3 0.3 0.3; visual box size=0.3 0.6 0.4
