Commit message: basic setup

File: urdf/plane_box.urdf (robot description, URDF)
Before this commit: robot simple_box, 1 links, 0 joints
Links:
- link box_link: mass 0.1 -> 1; geometry collision box size=5 5 0.01; visual box size=5 5 0.01

Commit message: update

File: urdf/plane_box.urdf (robot description, URDF)
Before this commit: robot plane_box, 1 links, 0 joints
Links:
- link box_link: geometry collision box size=5 5 0.001; visual box size=5 5 0.001
