Commit message: update

File: urdf/mobile_robot_with_arm.urdf (robot description, URDF)
Before this commit: robot mobile_robot_with_arm, 19 links, 18 joints
Links:
- link back_caster_link: geometry collision box size=0.08 0.08 0.08; visual box size=0.08 0.08 0.08
- link base_link: mass 10.0 -> 15.0; geometry collision box size=0.5 0.5 0.15; visual box size=0.5 0.5 0.15
- link bumper_link: geometry collision box size=0.015 0.5 0.15; visual box size=0.015 0.5 0.15
- link front_caster_link: geometry collision box size=0.08 0.08 0.08; visual box size=0.08 0.08 0.08
- link left_wheel_link: mass 2.0 -> 3.0; geometry collision cylinder length=0.04 radius=0.08; visual cylinder length=0.04 radius=0.08
- link right_wheel_link: mass 2.0 -> 3.0; geometry collision cylinder length=0.04 radius=0.08; visual cylinder length=0.04 radius=0.08
Joints:
- joint arm_base_mount_joint: origin xyz=0.0 0.0 0.05 rpy=0 0 0 -> xyz=0.0 0.0 0.075 rpy=0 0 0
- joint back_caster_joint: origin xyz=-0.09 0.0 -0.075 rpy=0 0 0 -> xyz=-0.15 0.0 -0.11 rpy=0 0 0
- joint bumper_joint: origin xyz=0.155 0.0 0.0 rpy=0 0 0 -> xyz=0.2575 0.0 0.0 rpy=0 0 0
- joint front_caster_joint: origin xyz=0.09 0.0 -0.075 rpy=0 0 0 -> xyz=0.15 0.0 -0.11 rpy=0 0 0
- joint left_wheel_joint: origin xyz=0.0 -0.1625 -0.05 rpy=0 0 0 -> xyz=0.0 -0.27 -0.075 rpy=0 0 0
- joint lidar_joint: origin xyz=0.0 0.0 0.065 rpy=0 0 0 -> xyz=0.0 0.0 0.0975 rpy=0 0 0
- joint rgbd_camera_joint: origin xyz=0.12 0.0 0.08 rpy=0 0 0 -> xyz=0.2 0.0 0.12 rpy=0 0 0
- joint right_wheel_joint: origin xyz=0.0 0.1625 -0.05 rpy=0 0 0 -> xyz=0.0 0.27 -0.075 rpy=0 0 0

Commit message: update

File: urdf/mobile_robot_with_arm.urdf (robot description, URDF)
Before this commit: robot mobile_robot_with_arm, 19 links, 18 joints
Links:
- removed link arm_base_link
- removed link gripper_left_link
- removed link gripper_right_link
- removed link link1
- removed link link2
- removed link link3
- removed link link4
- removed link link5
- removed link link6
- added link forearm_link, mass 2.275; collision mesh filename=ur5/collision/forearm.stl; visual mesh filename=ur5/visual/forearm.stl
- added link front_left_wheel_link, mass 3.0; collision cylinder length=0.04 radius=0.08; visual cylinder length=0.04 radius=0.08
- added link front_right_wheel_link, mass 3.0; collision cylinder length=0.04 radius=0.08; visual cylinder length=0.04 radius=0.08
- added link gripper_base_link, mass 0.001
- added link robotiq_2f_85_base, mass 0.1; visual mesh filename=gripper/robotiq-2f-base.obj scale=0.5 0.5 0.5
- added link robotiq_2f_85_left_coupler, mass 0.1; visual mesh filename=gripper/robotiq-2f-coupler.obj scale=0.5 0.5 0.5
- added link robotiq_2f_85_left_driver, mass 0.1; visual mesh filename=gripper/robotiq-2f-driver.obj scale=0.5 0.5 0.5
- added link robotiq_2f_85_left_follower, mass 0.1; collision mesh filename=gripper/robotiq-2f-follower.stl scale=0.005 0.005 0.005; visual mesh filename=gripper/robotiq-2f-follower.obj scale=0.5 0.5 0.5
- added link robotiq_2f_85_left_pad, mass 0.1; collision mesh filename=gripper/robotiq-2f-pad.stl scale=0.005 0.005 0.005; visual mesh filename=gripper/robotiq-2f-pad.stl scale=0.0005 0.0005 0.0005
- added link robotiq_2f_85_left_spring_link, mass 0.1; collision mesh filename=gripper/robotiq-2f-spring_link.stl scale=0.005 0.005 0.005; visual mesh filename=gripper/robotiq-2f-spring_link.obj scale=0.5 0.5 0.5
- added link robotiq_2f_85_right_coupler, mass 0.1; visual mesh filename=gripper/robotiq-2f-coupler.obj scale=0.5 0.5 0.5
- added link robotiq_2f_85_right_driver, mass 0.1; visual mesh filename=gripper/robotiq-2f-driver.obj scale=0.5 0.5 0.5
- added link robotiq_2f_85_right_follower, mass 0.1; collision mesh filename=gripper/robotiq-2f-follower.stl scale=0.005 0.005 0.005; visual mesh filename=gripper/robotiq-2f-follower.obj scale=0.5 0.5 0.5
- added link robotiq_2f_85_right_pad, mass 0.1; collision mesh filename=gripper/robotiq-2f-pad.stl scale=0.005 0.005 0.005; visual mesh filename=gripper/robotiq-2f-pad.stl scale=0.0005 0.0005 0.0005
- added link robotiq_2f_85_right_spring_link, mass 0.1; collision mesh filename=gripper/robotiq-2f-spring_link.stl scale=0.005 0.005 0.005; visual mesh filename=gripper/robotiq-2f-spring_link.obj scale=0.5 0.5 0.5
- added link shoulder_link, mass 3.7; collision mesh filename=ur5/collision/shoulder.stl; visual mesh filename=ur5/visual/shoulder.stl
- added link upper_arm_link, mass 8.393; collision mesh filename=ur5/collision/upperarm.stl; visual mesh filename=ur5/visual/upperarm.stl
- added link ur5_base_link, mass 4.0; collision mesh filename=ur5/collision/base.stl; visual mesh filename=ur5/visual/base.stl
- added link wrist_1_link, mass 1.219; collision mesh filename=ur5/collision/wrist1.stl; visual mesh filename=ur5/visual/wrist1.stl
- added link wrist_2_link, mass 1.219; collision mesh filename=ur5/collision/wrist2.stl; visual mesh filename=ur5/visual/wrist2.stl
- added link wrist_3_link, mass 0.1879; collision mesh filename=ur5/collision/wrist3.stl; visual mesh filename=ur5/visual/wrist3.stl
- link base_link: mass 15.0 -> 150.0; geometry collision box size=0.8 0.5 0.15; visual box size=0.8 0.5 0.15
Joints:
- removed joint arm_base_joint
- removed joint gripper_left_joint
- removed joint gripper_right_joint
- removed joint joint1
- removed joint joint2
- removed joint joint3
- removed joint joint4
- removed joint joint5
- removed joint joint6
- added joint elbow_joint: type revolute, parent upper_arm_link, child forearm_link, origin xyz=0.0 -0.1197 0.425 rpy=0.0 0.0 0.0, axis 0 1 0, limit lower=-3.14159265359 upper=3.14159265359 effort=150.0 velocity=3.15
- added joint front_left_wheel_joint: type continuous, parent base_link, child front_left_wheel_link, origin xyz=0.3 -0.27 -0.075 rpy=0 0 0, axis 0 1 0
- added joint front_right_wheel_joint: type continuous, parent base_link, child front_right_wheel_link, origin xyz=0.3 0.27 -0.075 rpy=0 0 0, axis 0 1 0
- added joint gripper_base_link_robotiq_2f_85_base_joint: type fixed, parent gripper_base_link, child robotiq_2f_85_base, origin xyz=0 0 0 rpy=0 0 0
- added joint robotiq_2f_85_left_coupler_joint: type fixed, parent robotiq_2f_85_left_driver, child robotiq_2f_85_left_coupler, origin xyz=0 0.1575 -0.0205 rpy=0 0 0
- added joint robotiq_2f_85_left_driver_joint: type revolute, parent robotiq_2f_85_base, child robotiq_2f_85_left_driver, origin xyz=0 -0.1530055 0.27452 rpy=0 0 3.141592653589793, axis 1 0 0, limit lower=0.0 upper=0.834 effort=60 velocity=1.91986177778
- added joint robotiq_2f_85_left_follower_joint: type revolute, parent robotiq_2f_85_left_coupler, child robotiq_2f_85_left_follower, origin xyz=0 0.0305 0.2355 rpy=0 0 0, axis 1 0 0, limit lower=-2.96705911111 upper=2.96705911111 effort=176 velocity=1.91986177778, mimic joint=robotiq_2f_85_right_driver_joint multiplier=-1
- added joint robotiq_2f_85_left_pad_joint: type fixed, parent robotiq_2f_85_left_follower, child robotiq_2f_85_left_pad
- added joint robotiq_2f_85_left_spring_link_joint: type revolute, parent robotiq_2f_85_base, child robotiq_2f_85_left_spring_link, origin xyz=0 -0.06 0.307 rpy=0 0 3.141592653589793, axis 1 0 0, limit lower=-2.96705911111 upper=2.96705911111 effort=176 velocity=1.91986177778, mimic joint=robotiq_2f_85_right_driver_joint multiplier=1
- added joint robotiq_2f_85_right_coupler_joint: type fixed, parent robotiq_2f_85_right_driver, child robotiq_2f_85_right_coupler, origin xyz=0 0.1575 -0.0205 rpy=0 0 0
- added joint robotiq_2f_85_right_driver_joint: type revolute, parent robotiq_2f_85_base, child robotiq_2f_85_right_driver, origin xyz=0 0.1530055 0.27452 rpy=0 0 0, axis 1 0 0, limit lower=0.0 upper=0.834 effort=60 velocity=1.91986177778
- added joint robotiq_2f_85_right_follower_joint: type revolute, parent robotiq_2f_85_right_coupler, child robotiq_2f_85_right_follower, origin xyz=0 0.0305 0.2355 rpy=0 0 0, axis 1 0 0, limit lower=-2.96705911111 upper=2.96705911111 effort=176 velocity=1.91986177778, mimic joint=robotiq_2f_85_right_driver_joint multiplier=-1
- added joint robotiq_2f_85_right_pad_joint: type fixed, parent robotiq_2f_85_right_follower, child robotiq_2f_85_right_pad
- added joint robotiq_2f_85_right_spring_link_joint: type revolute, parent robotiq_2f_85_base, child robotiq_2f_85_right_spring_link, origin xyz=0 0.06 0.307 rpy=0 0 0, axis 1 0 0, limit lower=-2.96705911111 upper=2.96705911111 effort=176 velocity=1.91986177778, mimic joint=robotiq_2f_85_right_driver_joint multiplier=1
- added joint shoulder_lift_joint: type revolute, parent shoulder_link, child upper_arm_link, origin xyz=0.0 0.13585 0.0 rpy=0.0 1.57079632679 0.0, axis 0 1 0, limit lower=-6.28318530718 upper=6.28318530718 effort=150.0 velocity=3.15
- added joint shoulder_pan_joint: type revolute, parent ur5_base_link, child shoulder_link, origin xyz=0.0 0.0 0.089159 rpy=0.0 0.0 0.0, axis 0 0 1, limit lower=-6.28318530718 upper=6.28318530718 effort=150.0 velocity=3.15
- added joint ur5_base_mount_joint: type fixed, parent arm_base_mount_link, child ur5_base_link, origin xyz=0.0 0.0 0.2 rpy=0 0 0
- added joint wrist_1_joint: type revolute, parent forearm_link, child wrist_1_link, origin xyz=0.0 0.0 0.39225 rpy=0.0 1.57079632679 0.0, axis 0 1 0, limit lower=-6.28318530718 upper=6.28318530718 effort=28.0 velocity=3.2
- added joint wrist_2_joint: type revolute, parent wrist_1_link, child wrist_2_link, origin xyz=0.0 0.093 0.0 rpy=0.0 0.0 0.0, axis 0 0 1, limit lower=-6.28318530718 upper=6.28318530718 effort=28.0 velocity=3.2
- added joint wrist_3_gripper_joint: type fixed, parent wrist_3_link, child gripper_base_link, origin xyz=0 0 0.0 rpy=0 0 0
- added joint wrist_3_joint: type revolute, parent wrist_2_link, child wrist_3_link, origin xyz=0.0 0.0 0.09465 rpy=0.0 0.0 0.0, axis 0 1 0, limit lower=-6.28318530718 upper=6.28318530718 effort=28.0 velocity=3.2
- joint back_caster_joint: origin xyz=-0.15 0.0 -0.11 rpy=0 0 0 -> xyz=-0.35 0.0 -0.11 rpy=0 0 0
- joint bumper_joint: origin xyz=0.2575 0.0 0.0 rpy=0 0 0 -> xyz=0.4075 0.0 0.0 rpy=0 0 0
- joint front_caster_joint: origin xyz=0.15 0.0 -0.11 rpy=0 0 0 -> xyz=0.35 0.0 -0.11 rpy=0 0 0
- joint left_wheel_joint: origin xyz=0.0 -0.27 -0.075 rpy=0 0 0 -> xyz=-0.3 -0.27 -0.075 rpy=0 0 0
- joint rgbd_camera_joint: origin xyz=0.2 0.0 0.12 rpy=0 0 0 -> xyz=0.4 0.0 0.12 rpy=0 0 0
- joint right_wheel_joint: origin xyz=0.0 0.27 -0.075 rpy=0 0 0 -> xyz=-0.3 0.27 -0.075 rpy=0 0 0

Commit message: update

File: urdf/mobile_robot_with_arm.urdf (robot description, URDF)
Before this commit: robot mobile_robot_with_arm, 31 links, 30 joints
Links:
- link robotiq_2f_85_right_follower: geometry collision mesh filename=gripper/robotiq-2f-follower.stl scale=0.025 0.025 0.025; visual mesh filename=gripper/robotiq-2f-follower.obj scale=0.5 0.5 0.5
- link robotiq_2f_85_right_pad: geometry collision mesh filename=gripper/robotiq-2f-pad.stl scale=0.025 0.025 0.025; visual mesh filename=gripper/robotiq-2f-pad.stl scale=0.0005 0.0005 0.0005
- link robotiq_2f_85_right_spring_link: geometry collision mesh filename=gripper/robotiq-2f-spring_link.stl scale=0.025 0.025 0.025; visual mesh filename=gripper/robotiq-2f-spring_link.obj scale=0.5 0.5 0.5

Commit message: Before madness

File: urdf/mobile_robot_with_arm.urdf (robot description, URDF)
Before this commit: robot mobile_robot_with_arm, 31 links, 30 joints
Links:
- link robotiq_2f_85_left_follower: geometry collision mesh filename=gripper/robotiq-2f-follower.stl scale=0.001 0.001 0.001; visual mesh filename=gripper/robotiq-2f-follower.obj scale=0.5 0.5 0.5
- link robotiq_2f_85_left_pad: geometry collision mesh filename=gripper/robotiq-2f-pad.stl scale=0.001 0.001 0.001; visual mesh filename=gripper/robotiq-2f-pad.stl scale=0.0005 0.0005 0.0005
- link robotiq_2f_85_left_spring_link: geometry collision mesh filename=gripper/robotiq-2f-spring_link.stl scale=0.001 0.001 0.001; visual mesh filename=gripper/robotiq-2f-spring_link.obj scale=0.5 0.5 0.5
- link robotiq_2f_85_right_follower: geometry collision mesh filename=gripper/robotiq-2f-follower.stl scale=0.005 0.005 0.005; visual mesh filename=gripper/robotiq-2f-follower.obj scale=0.5 0.5 0.5
- link robotiq_2f_85_right_pad: geometry collision mesh filename=gripper/robotiq-2f-pad.stl scale=0.005 0.005 0.005; visual mesh filename=gripper/robotiq-2f-pad.stl scale=0.0005 0.0005 0.0005
- link robotiq_2f_85_right_spring_link: geometry collision mesh filename=gripper/robotiq-2f-spring_link.stl scale=0.005 0.005 0.005; visual mesh filename=gripper/robotiq-2f-spring_link.obj scale=0.5 0.5 0.5
